Commit message: improve environment
improve environment 
*update reward
*change control to torque control

File: 2links.urdf (robot description, URDF)
Before this commit: robot 2rr, 4 links, 3 joints
Joints:
- joint R1: limit lower=0 upper=1.57 effort=0 velocity=0 -> lower=-0.523599 upper=0.523599 effort=300 velocity=12

Commit message: adding endEffector to end of arm

File: 2links.urdf (robot description, URDF)
Before this commit: robot 2rr, 4 links, 3 joints
Links:
- added link EndEffector, mass 0; visual cylinder length=0.30 radius=0.015
Joints:
- added joint r3: type fixed, parent arm, child EndEffector, origin xyz=0.0 -0.6 -0.15 rpy=0 0 -3.0804, axis 0 0 -1

File: goal.urdf (robot description, URDF)
Before this commit: robot goal, 1 links, 0 joints
Links:
- link base_link: geometry visual cylinder length=0.25 radius=0.055

Commit message: use resetJointState

File: 2links.urdf (robot description, URDF)
Before this commit: robot 2rr, 5 links, 4 joints
Joints:
- joint r2: limit lower=-1.57 upper=0 effort=0 velocity=0 -> lower=-1.57 upper=1.57 effort=0 velocity=0
